Commit message: Update URDF with sensors.
Signed-off-by: Benjamin Perseghetti <bperseghetti@rudislabs.com>

File: rdd2_description/urdf/rdd2.urdf (robot description, URDF)
Before this commit: robot rdd2, 2 links, 1 joints
Links:
- added link camera_link; visual box size=.008 .014 .01; visual box size=.008 .028 .028
- added link camera_link_optical
- added link lidar_link; visual box size=0.039 0.039 0.022; visual cylinder length=0.014 radius=0.018
Joints:
- added joint camera_joint: type fixed, parent base_link, child camera_link, origin xyz=.173 0 .145 rpy=0 0 0
- added joint camera_optical_joint: type fixed, parent camera_link, child camera_link_optical, origin xyz=.016 0 .006 rpy=-1.57079632679 0 -1.57079632679
- added joint lidar_joint: type fixed, parent base_link, child lidar_link, origin xyz=0 0 0.191 rpy=0 0 0
